File: eagle/th/th.brd (EAGLE design)
At the start: 67.8 x 61.7 mm, 54 parts

Commit message: add
Parts:
- removed C17: (no value), myparts:CAPACITOR-8-3.5
- C16: device myparts:CAPACITOR-8-3.5 -> myparts:CAPACITOR-10-5
- moved C16 2.05 mm to (62.5, 14.2), flipped to the bottom, turned to 90 degrees
Connections:
- removed net N$21: C16.P$2, C17.P$1
- net N$22: now also C16.P$2; no longer C17.P$2
Routing:
- net N$22: track 95.2 -> 104.0 mm
- net N$21: track 4.76 -> 0.00 mm
- net GND: track 59.0 -> 61.5 mm, vias 26 -> 29
Changed lines of the file:
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@@
 <attribute name="VALUE" x="34.29" y="14.859" size="1.016" layer="27" rot="R180"/>
-</element>
-<element name="C16" library="myparts" package="CAPACITOR-8-3.5" value="" x="60.579" y="14.986" smashed="yes" rot="R180">
-<attribute name="NAME" x="61.6505" y="10.738" size="0.8128" layer="25" rot="R180"/>
-<attribute name="VALUE" x="63.111" y="15.026" size="1.016" layer="27" rot="R180"/>
-</element>
-<element name="C17" library="myparts" package="CAPACITOR-8-3.5" value="" x="52.324" y="14.986" smashed="yes" rot="R180">
-<attribute name="NAME" x="53.3955" y="10.738" size="0.8128" layer="25" rot="R180"/>
-<attribute name="VALUE" x="54.856" y="15.026" size="1.016" layer="27" rot="R180"/>
 </element>
 <element name="CON2" library="myparts" package="HEADER-8P-2R-DIP-2_54MM" value="" x="24.003" y="57.531" smashed="yes" rot="MR0">
@@
 <element name="C15" library="myparts" package="0603" value="" x="44.704" y="29.591" smashed="yes">
 <attribute name="NAME" x="47.244" y="29.591" size="0.8128" layer="25" align="center"/>
+</element>
+<element name="C16" library="myparts" package="CAPACITOR-10-5" value="" x="62.484" y="14.224" smashed="yes" rot="MR90">
+<attribute name="NAME" x="62.414" y="11.7555" size="0.8128" layer="26" rot="MR90"/>
 </element>
 </elements>
@@
 <contactref element="BAT1" pad="2"/>
 <contactref element="IC1" pad="45"/>
-<via x="19.05" y="37.338" extent="1-16" drill="0.4"/>
 <via x="23.749" y="46.101" extent="1-16" drill="0.4"/>
 <via x="20.574" y="50.927" extent="1-16" drill="0.4"/>
@@
 <wire x1="21.336" y1="25.146" x2="21.336" y2="26.543" width="0.3048" layer="1"/>
 <wire x1="21.336" y1="26.543" x2="20.8915" y2="26.9875" width="0.3048" layer="1"/>
-<contactref element="C16" pad="P$1"/>
 <contactref element="SW2" pad="P$2"/>
 <contactref element="CON2" pad="4"/>
@@
 <wire x1="37.211" y1="7.493" x2="37.211" y2="8.89" width="0.6096" layer="1"/>
 <wire x1="38.735" y1="7.62" x2="38.735" y2="8.89" width="0.6096" layer="1"/>
+<via x="17.272" y="39.116" extent="1-16" drill="0.4"/>
+<via x="20.828" y="39.116" extent="1-16" drill="0.4"/>
+<via x="20.828" y="35.56" extent="1-16" drill="0.4"/>
+<contactref element="C16" pad="P$1"/>
+<via x="17.272" y="35.56" extent="1-16" drill="0.4"/>
+<wire x1="19.05" y1="37.338" x2="20.828" y2="35.56" width="0.3048" layer="1"/>
 </signal>
 <signal name="N$2">
@@
 <via x="8.763" y="24.511" extent="1-16" drill="0.4"/>
 <wire x1="9.906" y1="24.511" x2="8.763" y2="24.511" width="0.3048" layer="1"/>
-<wire x1="5.715" y1="24.511" x2="1.524" y2="24.511" width="0.3048" layer="1"/>
+<wire x1="5.715" y1="24.511" x2="1.524" y2="23.241" width="0.3048" layer="1"/>
 <wire x1="5.715" y1="24.511" x2="8.763" y2="24.511" width="0.3048" layer="16"/>
 </signal>
@@
 <wire x1="53.975" y1="34.925" x2="60.96" y2="34.925" width="1.778" layer="1"/>
 </signal>
-<signal name="N$21">
-<contactref element="C16" pad="P$2"/>
-<contactref element="C17" pad="P$1"/>
-<wire x1="54.074" y1="14.986" x2="58.829" y2="14.986" width="1.778" layer="1"/>
-</signal>
 <signal name="GND1">
 <polygon width="0.0508" layer="16" pour="cutout">
@@
 <contactref element="C12" pad="2"/>
 <contactref element="C13" pad="2"/>
-<contactref element="C17" pad="P$2"/>
 <contactref element="C14" pad="2"/>
 <contactref element="C15" pad="2"/>
@@
 <wire x1="46.736" y1="34.163" x2="49.53" y2="34.163" width="1.778" layer="16"/>
 <wire x1="49.53" y1="49.149" x2="49.53" y2="34.163" width="1.778" layer="1"/>
-<wire x1="49.53" y1="34.163" x2="49.53" y2="16.03" width="1.778" layer="1"/>
-<wire x1="49.53" y1="16.03" x2="50.574" y2="14.986" width="1.778" layer="1"/>
 <wire x1="27.94" y1="49.149" x2="27.94" y2="49.276" width="0.6096" layer="1"/>
 <wire x1="27.94" y1="49.276" x2="26.9748" y2="50.2412" width="0.6096" layer="1"/>
@@
 <wire x1="20.193" y1="56.84400625" x2="20.193" y2="56.388" width="0.6096" layer="1"/>
 <wire x1="20.193" y1="58.801" x2="20.193" y2="56.84400625" width="0.3048" layer="1"/>
+<contactref element="C16" pad="P$2"/>
+<wire x1="49.53" y1="34.163" x2="49.53" y2="20.066" width="1.778" layer="1"/>
+<wire x1="52.832" y1="16.764" x2="62.484" y2="16.764" width="1.778" layer="1"/>
+<wire x1="49.53" y1="20.066" x2="52.832" y2="16.764" width="1.778" layer="1"/>
 </signal>
 <signal name="N$14">

Commit message: add
Parts:
- removed C21: (no value), myparts:0603
- added C17: (no value), myparts:0603
- moved C19 31.3 mm to (30.9, 17.7)
- moved C18 24.8 mm to (22.0, 47.6), turned to 180 degrees
- moved C20 3.05 mm to (30.9, 14.6)
Connections:
- net GND: now also C17.1; no longer C21.1
- net N$14: now also C20.2; no longer C21.2
- net N$2: now also C17.2; no longer C18.2
- net N$20: now also C18.2; no longer C19.2
- net N$25: now also C19.2; no longer C20.2
Routing:
- net N$9: track 33.7 -> 38.5 mm
- net N$1: track 103.7 -> 106.8 mm
- net N$8: track 34.7 -> 33.4 mm
Changed lines of the file:
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@@
 <attribute name="NAME" x="47.244" y="32.639" size="0.8128" layer="25" align="center"/>
 </element>
-<element name="C18" library="myparts" package="0603" value="" x="41.783" y="32.639" smashed="yes">
+<element name="C17" library="myparts" package="0603" value="" x="41.783" y="32.639" smashed="yes">
 <attribute name="NAME" x="40.005" y="32.766" size="0.8128" layer="25" rot="R90" align="center"/>
 </element>
-<element name="C19" library="myparts" package="0603" value="" x="21.971" y="47.625" smashed="yes" rot="R180">
+<element name="C18" library="myparts" package="0603" value="" x="21.971" y="47.625" smashed="yes" rot="R180">
 <attribute name="NAME" x="24.511" y="47.625" size="0.8128" layer="25" rot="R180" align="center"/>
 </element>
@@
 <attribute name="VALUE" x="34.29" y="19.431" size="1.016" layer="27" rot="R180"/>
 </element>
-<element name="C20" library="myparts" package="0603" value="" x="30.861" y="17.653" smashed="yes" rot="R180">
+<element name="C19" library="myparts" package="0603" value="" x="30.861" y="17.653" smashed="yes" rot="R180">
 <attribute name="NAME" x="28.321" y="17.653" size="0.8128" layer="25" rot="R180" align="center"/>
 <attribute name="VALUE" x="34.29" y="17.907" size="1.016" layer="27" rot="R180"/>
 </element>
-<element name="C21" library="myparts" package="0603" value="" x="30.861" y="14.605" smashed="yes" rot="R180">
+<element name="C20" library="myparts" package="0603" value="" x="30.861" y="14.605" smashed="yes" rot="R180">
 <attribute name="NAME" x="28.321" y="14.605" size="0.8128" layer="25" rot="R180" align="center"/>
 <attribute name="VALUE" x="34.29" y="14.859" size="1.016" layer="27" rot="R180"/>
@@
 <signals>
 <signal name="GND">
-<contactref element="C18" pad="1"/>
+<contactref element="C17" pad="1"/>
 <contactref element="C12" pad="1"/>
 <contactref element="CON1" pad="6"/>
@@
 <contactref element="C6" pad="1"/>
 <contactref element="R16" pad="1"/>
-<contactref element="C19" pad="1"/>
+<contactref element="C18" pad="1"/>
 <contactref element="Q1" pad="1"/>
 <via x="16.637" y="31.242" extent="1-16" drill="0.4"/>
@@
 <contactref element="CON5" pad="2"/>
 <contactref element="R13" pad="1"/>
+<contactref element="C19" pad="1"/>
 <contactref element="C20" pad="1"/>
-<contactref element="C21" pad="1"/>
 <wire x1="17.05" y1="40.767" x2="17.05" y2="42.767" width="0.3048" layer="1"/>
 <wire x1="17.05" y1="42.767" x2="17.018" y2="42.799" width="0.3048" layer="1"/>
@@
 <signal name="N$2">
 <contactref element="R10" pad="1"/>
-<contactref element="C18" pad="2"/>
+<contactref element="C17" pad="2"/>
 <contactref element="R9" pad="1"/>
 <contactref element="MOD1" pad="18"/>
@@
 <wire x1="14.002" y1="35.338" x2="13.335" y2="34.671" width="0.3048" layer="1"/>
 <wire x1="13.335" y1="34.671" x2="13.208" y2="34.671" width="0.3048" layer="1"/>
-<wire x1="7.874" y1="38.738725" x2="8.382" y2="38.230725" width="0.3048" layer="1"/>
-<wire x1="8.382" y1="36.40915" x2="10.37415" y2="34.417" width="0.3048" layer="1"/>
 <wire x1="12.954" y1="34.671" x2="13.208" y2="34.671" width="0.3048" layer="1"/>
-<wire x1="12.954" y1="34.671" x2="12.7" y2="34.417" width="0.3048" layer="1"/>
-<wire x1="12.7" y1="34.417" x2="10.37415" y2="34.417" width="0.3048" layer="1"/>
-<wire x1="8.382" y1="38.230725" x2="8.382" y2="36.40915" width="0.3048" layer="1"/>
+<wire x1="12.7" y1="34.417" x2="12.954" y2="34.671" width="0.3048" layer="1"/>
 <wire x1="10.033" y1="56.892275" x2="7.874" y2="54.733275" width="0.3048" layer="1"/>
-<wire x1="7.874" y1="54.733275" x2="7.874" y2="38.738725" width="0.3048" layer="1"/>
+<wire x1="6.35" y1="34.163" x2="7.239" y2="33.274" width="0.3048" layer="1"/>
+<wire x1="7.239" y1="33.274" x2="9.017" y2="33.274" width="0.3048" layer="1"/>
+<wire x1="10.16" y1="34.417" x2="12.7" y2="34.417" width="0.3048" layer="1"/>
+<wire x1="7.874" y1="54.733275" x2="7.874" y2="37.211" width="0.3048" layer="1"/>
+<wire x1="7.874" y1="37.211" x2="6.35" y2="35.687" width="0.3048" layer="1"/>
+<wire x1="6.35" y1="35.687" x2="6.35" y2="34.163" width="0.3048" layer="1"/>
+<wire x1="9.017" y1="33.274" x2="10.16" y2="34.417" width="0.3048" layer="1"/>
 </signal>
 <signal name="N$10">
@@
 <via x="5.969" y="38.227" extent="1-16" drill="0.7"/>
 <wire x1="5.969" y1="38.227" x2="12.192" y2="38.227" width="0.8128" layer="16"/>
-<wire x1="4.318" y1="33.655" x2="7.239" y2="30.734" width="1.778" layer="1"/>
-<wire x1="5.969" y1="38.227" x2="4.318" y2="36.576" width="1.778" layer="1"/>
-<wire x1="4.318" y1="36.576" x2="4.318" y2="33.655" width="1.778" layer="1"/>
-<wire x1="7.239" y1="30.734" x2="7.239" y2="23.241" width="1.778" layer="1"/>
+<wire x1="4.445" y1="33.401" x2="7.239" y2="30.607" width="1.778" layer="1"/>
+<wire x1="5.969" y1="38.227" x2="4.445" y2="36.703" width="1.778" layer="1"/>
+<wire x1="4.445" y1="36.703" x2="4.445" y2="33.401" width="1.778" layer="1"/>
+<wire x1="7.239" y1="30.607" x2="7.239" y2="23.241" width="1.778" layer="1"/>
 <wire x1="32.766" y1="7.62" x2="35.306" y2="7.62" width="0.6096" layer="1"/>
 <wire x1="35.306" y1="7.62" x2="35.433" y2="7.493" width="0.6096" layer="1"/>
@@
 <wire x1="39.171" y1="54.483" x2="40.06" y2="54.483" width="0.3048" layer="16"/>
 <wire x1="38.735" y1="60.579" x2="38.735" y2="53.467" width="0.3048" layer="1"/>
-<wire x1="7.366" y1="38.5283" x2="7.874" y2="38.0203" width="0.3048" layer="1"/>
-<wire x1="7.874" y1="38.0203" x2="7.874" y2="36.198725" width="0.3048" layer="1"/>
 <wire x1="10.414" y1="25.019" x2="9.906" y2="24.511" width="0.3048" layer="1"/>
 <wire x1="10.414" y1="25.019" x2="10.414" y2="27.432" width="0.3048" layer="1"/>
 <wire x1="10.414" y1="28.956" x2="9.398" y2="28.956" width="0.3048" layer="1"/>
-<wire x1="8.636" y1="29.718" x2="8.636" y2="32.258" width="0.3048" layer="1"/>
 <wire x1="9.398" y1="28.956" x2="8.636" y2="29.718" width="0.3048" layer="1"/>
-<wire x1="7.874" y1="36.198725" x2="8.636" y2="35.436725" width="0.3048" layer="1"/>
-<wire x1="8.636" y1="35.436725" x2="8.636" y2="33.147" width="0.3048" layer="1"/>
-<wire x1="8.636" y1="33.147" x2="8.636" y2="32.258" width="0.3048" layer="1"/>
 <wire x1="16.764" y1="32.512" x2="13.51910625" y2="32.512" width="0.3048" layer="1"/>
 <wire x1="13.51910625" y1="32.512" x2="13.13490625" y2="32.8962" width="0.3048" layer="1"/>
 <wire x1="13.13490625" y1="32.8962" x2="12.89369375" y2="32.8962" width="0.3048" layer="1"/>
-<wire x1="12.64289375" y1="33.147" x2="8.636" y2="33.147" width="0.3048" layer="1"/>
-<wire x1="12.89369375" y1="32.8962" x2="12.64289375" y2="33.147" width="0.3048" layer="1"/>
+<wire x1="12.64289375" y1="33.147" x2="12.89369375" y2="32.8962" width="0.3048" layer="1"/>
 <wire x1="25.781" y1="49.911" x2="25.781" y2="48.895" width="0.3048" layer="16"/>
 <wire x1="25.781" y1="48.895" x2="23.876" y2="46.99" width="0.3048" layer="16"/>
@@
 <wire x1="38.227" y1="51.181" x2="38.735" y2="51.689" width="0.3048" layer="16"/>
 <wire x1="7.366" y1="54.9437" x2="7.366" y2="42.926" width="0.3048" layer="1"/>
-<wire x1="7.366" y1="42.926" x2="7.366" y2="38.5283" width="0.3048" layer="1"/>
 <wire x1="8.763" y1="56.3407" x2="7.366" y2="54.9437" width="0.3048" layer="1"/>
 <via x="12.827" y="44.323" extent="1-16" drill="0.4"/>
@@
 <via x="8.763" y="24.511" extent="1-16" drill="0.4"/>
 <wire x1="9.906" y1="24.511" x2="8.763" y2="24.511" width="0.3048" layer="1"/>
-<wire x1="5.715" y1="24.511" x2="1.524" y2="23.241" width="0.3048" layer="1"/>
 <wire x1="5.715" y1="24.511" x2="8.763" y2="24.511" width="0.3048" layer="16"/>
+<wire x1="7.366" y1="37.421425" x2="5.842" y2="35.897425" width="0.3048" layer="1"/>
+<wire x1="5.842" y1="35.897425" x2="5.842" y2="33.952575" width="0.3048" layer="1"/>
+<wire x1="5.842" y1="33.952575" x2="7.028575" y2="32.766" width="0.3048" layer="1"/>
+<wire x1="7.366" y1="42.926" x2="7.366" y2="37.421425" width="0.3048" layer="1"/>
+<wire x1="9.608425" y1="33.147" x2="12.64289375" y2="33.147" width="0.3048" layer="1"/>
+<wire x1="7.028575" y1="32.766" x2="8.636" y2="32.766" width="0.3048" layer="1"/>
+<wire x1="8.636" y1="32.766" x2="9.227425" y2="32.766" width="0.3048" layer="1"/>
+<wire x1="9.227425" y1="32.766" x2="9.608425" y2="33.147" width="0.3048" layer="1"/>
+<wire x1="8.636" y1="29.718" x2="8.636" y2="32.766" width="0.3048" layer="1"/>
+<wire x1="5.715" y1="24.511" x2="5.715" y2="23.749" width="0.3048" layer="1"/>
+<wire x1="5.207" y1="23.241" x2="1.524" y2="23.241" width="0.3048" layer="1"/>
+<wire x1="5.715" y1="23.749" x2="5.207" y2="23.241" width="0.3048" layer="1"/>
 </signal>
 <signal name="N$5">
@@
 <wire x1="51.689" y1="32.639" x2="53.975" y2="34.925" width="1.778" layer="1"/>
 <wire x1="47.371" y1="26.797" x2="51.689" y2="26.797" width="1.778" layer="16"/>
-<wire x1="53.975" y1="34.925" x2="60.96" y2="34.925" width="1.778" layer="1"/>
+<wire x1="53.975" y1="34.925" x2="59.69" y2="34.925" width="1.778" layer="1"/>
 </signal>
 <signal name="GND1">
@@
 <contactref element="R16" pad="2"/>
 <contactref element="R15" pad="2"/>
-<contactref element="C19" pad="2"/>
+<contactref element="C18" pad="2"/>
 <contactref element="IC1" pad="37"/>
 <wire x1="21.209" y1="47.625" x2="21.209" y2="46.101" width="0.3048" layer="1"/>
@@
 <contactref element="R13" pad="2"/>
 <contactref element="CON5" pad="5"/>
-<contactref element="C21" pad="2"/>
+<contactref element="C20" pad="2"/>
 <wire x1="30.099" y1="16.129" x2="30.099" y2="14.605" width="0.3048" layer="1"/>
 <via x="24.511" y="31.242" extent="1-16" drill="0.4"/>
@@
 <contactref element="R14" pad="2"/>
 <contactref element="CON5" pad="6"/>
-<contactref element="C20" pad="2"/>
+<contactref element="C19" pad="2"/>
 <wire x1="30.099" y1="19.177" x2="30.099" y2="17.653" width="0.3048" layer="1"/>
 <via x="25.527" y="31.242" extent="1-16" drill="0.4"/>
