File: eagle/th/th.brd (EAGLE design)
At the start: 67.8 x 61.7 mm, 53 parts

Commit message: init
Parts:
- added D2: (no value), myparts:SOD123-DIODE
- added Q2: (no value), myparts:SOT23-3
- added R17, R18, R19: (no value), myparts:0603
- moved Q1 4.83 mm to (50.2, 6.48)
Connections:
- new net N$21: D2.1, Q2.1, R17.2, R18.2
- new net N$26: Q1.2, Q2.2, R19.2
- net GND: now also D2.2, R18.1
- net UVCC: now also R17.1
- net VCC: now also Q2.3, R19.1; no longer Q1.2
Routing:
- net UVCC: track 81.3 -> 104.2 mm
- net N$26: track 0.00 -> 10.2 mm
- net N$21: track 0.00 -> 6.33 mm
- net N$5: track 3.17 -> 7.33 mm
- net GND: track 61.5 -> 63.7 mm, vias 29 -> 31
Changed lines of the file:
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@@
 </element>
 <element name="C9" library="myparts" package="0805" value="" x="36.322" y="5.588" smashed="yes" rot="R180">
-<attribute name="NAME" x="38.847" y="4.93" size="0.8128" layer="25" rot="R180" align="center"/>
+<attribute name="NAME" x="38.593" y="4.549" size="0.8128" layer="25" rot="R270" align="center"/>
 </element>
 <element name="C10" library="myparts" package="0603" value="" x="39.497" y="7.62" smashed="yes">
-<attribute name="NAME" x="42.037" y="7.62" size="0.8128" layer="25" align="center"/>
+<attribute name="NAME" x="39.878" y="8.89" size="0.8128" layer="25" align="center"/>
 </element>
 <element name="C11" library="myparts" package="0603" value="" x="39.497" y="6.096" smashed="yes">
-<attribute name="NAME" x="42.037" y="6.096" size="0.8128" layer="25" align="center"/>
+<attribute name="NAME" x="40.005" y="4.953" size="0.8128" layer="25" align="center"/>
 </element>
 <element name="C2" library="myparts" package="0603" value="" x="11.176" y="30.48" smashed="yes">
@@
 <attribute name="VALUE" x="20.647" y="6.502" size="1.27" layer="27" rot="R180" align="center"/>
 </element>
-<element name="Q1" library="myparts" package="SOT23-3" value="" x="45.339" y="6.477" smashed="yes" rot="R90">
-<attribute name="NAME" x="45.339" y="8.89" size="0.8128" layer="25" rot="R180" align="center"/>
-<attribute name="VALUE" x="45.339" y="6.477" size="1.27" layer="27" rot="R90" align="center"/>
+<element name="Q1" library="myparts" package="SOT23-3" value="" x="50.165" y="6.477" smashed="yes" rot="R90">
+<attribute name="NAME" x="50.165" y="8.89" size="0.8128" layer="25" rot="R180" align="center"/>
+<attribute name="VALUE" x="50.165" y="6.477" size="1.27" layer="27" rot="R90" align="center"/>
 </element>
 <element name="R10" library="myparts" package="0603" value="" x="41.783" y="34.163" smashed="yes" rot="R180">
@@
 <element name="C16" library="myparts" package="CAPACITOR-10-5" value="" x="62.484" y="14.224" smashed="yes" rot="MR90">
 <attribute name="NAME" x="62.414" y="11.7555" size="0.8128" layer="26" rot="MR90"/>
+</element>
+<element name="R17" library="myparts" package="0603" value="" x="45.085" y="2.159" smashed="yes" rot="R180">
+<attribute name="NAME" x="47.625" y="2.159" size="0.8128" layer="25" rot="R180" align="center"/>
+</element>
+<element name="R18" library="myparts" package="0603" value="" x="45.085" y="3.683" smashed="yes" rot="R180">
+<attribute name="NAME" x="47.625" y="3.683" size="0.8128" layer="25" rot="R180" align="center"/>
+</element>
+<element name="Q2" library="myparts" package="SOT23-3" value="" x="45.085" y="6.477" smashed="yes" rot="R90">
+<attribute name="NAME" x="45.085" y="8.89" size="0.8128" layer="25" rot="R180" align="center"/>
+</element>
+<element name="D2" library="myparts" package="SOD123-DIODE" value="" x="42.164" y="5.842" smashed="yes" rot="R90">
+<attribute name="NAME" x="42.1255" y="8.8805" size="0.8128" layer="25" rot="R180" align="center"/>
+</element>
+<element name="R19" library="myparts" package="0603" value="" x="47.625" y="6.985" smashed="yes" rot="R270">
+<attribute name="NAME" x="47.625" y="9.525" size="0.8128" layer="25" rot="R270" align="center"/>
 </element>
 </elements>
@@
 <via x="24.511" y="34.925" extent="1-16" drill="0.4"/>
 <via x="11.176" y="36.195" extent="1-16" drill="0.4"/>
-<via x="44.45" y="3.683" extent="1-16" drill="0.7"/>
-<wire x1="44.389" y1="5.334" x2="44.389" y2="3.744" width="0.6096" layer="1"/>
-<wire x1="44.389" y1="3.744" x2="44.45" y2="3.683" width="0.381" layer="1"/>
+<via x="49.276" y="3.683" extent="1-16" drill="0.7"/>
+<wire x1="49.215" y1="5.334" x2="49.215" y2="3.744" width="0.6096" layer="1"/>
+<wire x1="49.215" y1="3.744" x2="49.276" y2="3.683" width="0.381" layer="1"/>
 <polygon width="0.254" layer="16">
 <vertex x="5.969" y="2.159"/>
@@
 <via x="17.272" y="35.56" extent="1-16" drill="0.4"/>
 <wire x1="19.05" y1="37.338" x2="20.828" y2="35.56" width="0.3048" layer="1"/>
+<contactref element="R18" pad="1"/>
+<contactref element="D2" pad="2"/>
+<via x="42.164" y="6.604" extent="1-16" drill="0.4"/>
+<wire x1="42.164" y1="7.6835" x2="42.164" y2="6.604" width="0.6096" layer="1"/>
+<via x="46.99" y="3.683" extent="1-16" drill="0.4"/>
+<wire x1="45.847" y1="3.683" x2="46.99" y2="3.683" width="0.6096" layer="1"/>
 </signal>
 <signal name="N$2">
@@
 <wire x1="33.02" y1="19.177" x2="33.02" y2="17.653" width="0.3048" layer="1"/>
 <contactref element="CON2" pad="3"/>
-<contactref element="Q1" pad="2"/>
 <wire x1="40.259" y1="10.795" x2="40.259" y2="19.812" width="1.778" layer="1"/>
 <wire x1="26.162" y1="48.387" x2="26.162" y2="48.895" width="1.778" layer="1"/>
@@
 <wire x1="31.877" y1="21.971" x2="31.877" y2="30.48" width="1.778" layer="1"/>
 <wire x1="40.259" y1="7.62" x2="40.259" y2="6.096" width="0.6096" layer="1"/>
-<wire x1="40.259" y1="7.62" x2="40.259" y2="10.795" width="0.6096" layer="1"/>
-<wire x1="46.289" y1="5.334" x2="46.289" y2="3.617" width="0.6096" layer="1"/>
-<wire x1="45.212" y1="2.54" x2="43.561" y2="2.54" width="0.6096" layer="1"/>
-<wire x1="43.561" y1="2.54" x2="42.672" y2="3.429" width="0.6096" layer="1"/>
-<wire x1="46.289" y1="3.617" x2="45.212" y2="2.54" width="0.6096" layer="1"/>
-<wire x1="42.672" y1="3.429" x2="40.259" y2="3.429" width="0.6096" layer="1"/>
-<wire x1="40.259" y1="3.429" x2="37.4015" y2="3.429" width="0.6096" layer="1"/>
-<wire x1="40.259" y1="6.096" x2="40.259" y2="3.429" width="0.6096" layer="1"/>
+<wire x1="40.259" y1="7.62" x2="40.259" y2="8.89" width="0.6096" layer="1"/>
+<wire x1="40.259" y1="8.89" x2="40.259" y2="10.795" width="0.6096" layer="1"/>
 <wire x1="33.02" y1="19.177" x2="32.893" y2="19.304" width="0.3048" layer="1"/>
 <wire x1="32.893" y1="19.304" x2="32.893" y2="20.955" width="0.3048" layer="1"/>
+<contactref element="Q2" pad="3"/>
+<contactref element="R19" pad="1"/>
+<wire x1="37.4015" y1="3.429" x2="39.624" y2="3.429" width="0.6096" layer="1"/>
+<wire x1="40.259" y1="4.064" x2="40.259" y2="6.096" width="0.6096" layer="1"/>
+<wire x1="39.624" y1="3.429" x2="40.259" y2="4.064" width="0.6096" layer="1"/>
+<wire x1="45.085" y1="7.62" x2="45.212" y2="7.747" width="0.6096" layer="1"/>
+<wire x1="45.212" y1="7.747" x2="47.625" y2="7.747" width="0.6096" layer="1"/>
+<wire x1="45.085" y1="7.62" x2="45.085" y2="8.509" width="0.6096" layer="1"/>
+<wire x1="44.704" y1="8.89" x2="40.259" y2="8.89" width="0.6096" layer="1"/>
+<wire x1="45.085" y1="8.509" x2="44.704" y2="8.89" width="0.6096" layer="1"/>
 </signal>
 <signal name="N$3">
@@
 <wire x1="21.082" y1="18.796" x2="21.082" y2="14.732" width="1.778" layer="1"/>
 <wire x1="24.13" y1="8.763" x2="25.4" y2="7.493" width="1.778" layer="1"/>
-<wire x1="29.972" y1="7.493" x2="25.4" y2="7.493" width="1.778" layer="1"/>
+<wire x1="29.972" y1="7.493" x2="28.956" y2="7.493" width="1.778" layer="1"/>
+<wire x1="28.956" y1="7.493" x2="25.4" y2="7.493" width="1.778" layer="1"/>
 <wire x1="9.779" y1="20.701" x2="19.177" y2="20.701" width="1.778" layer="1"/>
 <wire x1="21.082" y1="14.732" x2="24.13" y2="11.684" width="1.778" layer="1"/>
@@
 <wire x1="32.766" y1="7.62" x2="32.639" y2="7.493" width="0.6096" layer="1"/>
 <wire x1="32.639" y1="7.493" x2="29.972" y2="7.493" width="0.6096" layer="1"/>
+<contactref element="R17" pad="1"/>
+<wire x1="45.847" y1="2.159" x2="45.847" y2="1.27" width="0.6096" layer="1"/>
+<wire x1="45.847" y1="1.27" x2="45.593" y2="1.016" width="0.6096" layer="1"/>
+<wire x1="45.593" y1="1.016" x2="43.307" y2="1.016" width="0.6096" layer="1"/>
+<wire x1="43.307" y1="1.016" x2="42.418" y2="1.905" width="0.6096" layer="1"/>
+<wire x1="42.418" y1="1.905" x2="30.607" y2="1.905" width="0.6096" layer="1"/>
+<wire x1="28.956" y1="3.556" x2="28.956" y2="7.493" width="0.6096" layer="1"/>
+<wire x1="30.607" y1="1.905" x2="28.956" y2="3.556" width="0.6096" layer="1"/>
 </signal>
 <signal name="N$34">
@@
 <contactref element="Q1" pad="3"/>
 <contactref element="J1" pad="1"/>
-<wire x1="45.339" y1="7.62" x2="45.339" y2="10.795" width="0.6096" layer="1"/>
+<wire x1="50.165" y1="7.62" x2="50.165" y2="9.652" width="0.6096" layer="1"/>
+<wire x1="49.022" y1="10.795" x2="45.339" y2="10.795" width="0.6096" layer="1"/>
+<wire x1="50.165" y1="9.652" x2="49.022" y2="10.795" width="0.6096" layer="1"/>
 </signal>
 <signal name="N$8">
@@
 <wire x1="10.16" y1="42.291" x2="9.398" y2="41.529" width="0.3048" layer="1"/>
 </signal>
+<signal name="N$21">
+<contactref element="R17" pad="2"/>
+<contactref element="R18" pad="2"/>
+<contactref element="D2" pad="1"/>
+<contactref element="Q2" pad="1"/>
+<wire x1="44.135" y1="5.334" x2="44.135" y2="4.506" width="0.6096" layer="1"/>
+<wire x1="44.135" y1="4.506" x2="44.323" y2="4.318" width="0.6096" layer="1"/>
+<wire x1="44.323" y1="4.318" x2="44.323" y2="3.683" width="0.6096" layer="1"/>
+<wire x1="42.164" y1="4.0005" x2="42.164" y2="4.953" width="0.6096" layer="1"/>
+<wire x1="42.545" y1="5.334" x2="44.135" y2="5.334" width="0.6096" layer="1"/>
+<wire x1="42.164" y1="4.953" x2="42.545" y2="5.334" width="0.6096" layer="1"/>
+<wire x1="44.323" y1="3.683" x2="44.323" y2="2.159" width="0.6096" layer="1"/>
+</signal>
+<signal name="N$26">
+<contactref element="Q1" pad="2"/>
+<contactref element="Q2" pad="2"/>
+<contactref element="R19" pad="2"/>
+<wire x1="47.625" y1="6.223" x2="47.625" y2="5.334" width="0.6096" layer="1"/>
+<wire x1="47.625" y1="5.334" x2="47.625" y2="4.572" width="0.6096" layer="1"/>
+<wire x1="47.625" y1="4.572" x2="48.006" y2="4.191" width="0.6096" layer="1"/>
+<wire x1="48.006" y1="4.191" x2="48.006" y2="3.302" width="0.6096" layer="1"/>
+<wire x1="48.768" y1="2.54" x2="49.911" y2="2.54" width="0.6096" layer="1"/>
+<wire x1="49.911" y1="2.54" x2="51.115" y2="3.744" width="0.6096" layer="1"/>
+<wire x1="51.115" y1="3.744" x2="51.115" y2="5.334" width="0.6096" layer="1"/>
+<wire x1="48.006" y1="3.302" x2="48.768" y2="2.54" width="0.6096" layer="1"/>
+<wire x1="46.035" y1="5.334" x2="47.625" y2="5.334" width="0.6096" layer="1"/>
+</signal>
 </signals>
