File: eagle/th/th.sch (EAGLE design)
At the start: 54 parts

Commit message: add
Parts:
- removed C17: (no value), myparts:CAPACITOR-8-3.5
- C16: device myparts:CAPACITOR-8-3.5 -> myparts:CAPACITOR-10-5
Connections:
- removed net N$21: C16.2, C17.1
- net N$22: now also C16.2; no longer C17.2
Other:
- moved on the sheet: C16
Changed lines of the file:
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@@
 <part name="SUP7" library="myparts" deviceset="VCC" device=""/>
 <part name="SUP9" library="myparts" deviceset="VCC" device=""/>
-<part name="C16" library="myparts" deviceset="CAPACITOR-8-3.5" device=""/>
-<part name="C17" library="myparts" deviceset="CAPACITOR-8-3.5" device=""/>
 <part name="GND31" library="myparts" deviceset="GND" device=""/>
 <part name="GND13" library="myparts" deviceset="GND" device=""/>
@@
 <part name="GND14" library="myparts" deviceset="GND" device=""/>
 <part name="GND29" library="myparts" deviceset="GND" device=""/>
+<part name="C16" library="myparts" deviceset="CAPACITOR-10-5" device=""/>
 </parts>
 <sheets>
@@
 <attribute name="VALUE" x="-88.265" y="-10.795" size="1.778" layer="96"/>
 </instance>
-<instance part="C16" gate="G$1" x="180.34" y="2.54" smashed="yes" rot="R90">
-<attribute name="NAME" x="179.324" y="2.794" size="1.778" layer="95" rot="R90" align="center-left"/>
-<attribute name="VALUE" x="175.514" y="6.35" size="1.778" layer="96" rot="R90" align="center-left"/>
-</instance>
-<instance part="C17" gate="G$1" x="180.34" y="15.24" smashed="yes" rot="R90">
-<attribute name="NAME" x="179.324" y="15.494" size="1.778" layer="95" rot="R90" align="center-left"/>
-<attribute name="VALUE" x="175.514" y="19.05" size="1.778" layer="96" rot="R90" align="center-left"/>
-</instance>
-<instance part="GND31" gate="1" x="180.34" y="0" smashed="yes">
-<attribute name="VALUE" x="177.8" y="-3.048" size="1.778" layer="96"/>
+<instance part="GND31" gate="1" x="180.34" y="12.7" smashed="yes">
+<attribute name="VALUE" x="177.8" y="9.652" size="1.778" layer="96"/>
 </instance>
 <instance part="GND13" gate="1" x="-48.26" y="-63.5" smashed="yes">
@@
 <instance part="GND29" gate="1" x="175.26" y="12.7" smashed="yes">
 <attribute name="VALUE" x="172.72" y="9.652" size="1.778" layer="96"/>
+</instance>
+<instance part="C16" gate="G$1" x="180.34" y="15.24" smashed="yes" rot="R90">
+<attribute name="NAME" x="177.292" y="19.05" size="1.778" layer="95" rot="R90" align="center-left"/>
+<attribute name="VALUE" x="175.514" y="19.05" size="1.778" layer="96" rot="R90" align="center-left"/>
 </instance>
 </instances>
@@
 </segment>
 <segment>
-<pinref part="C16" gate="G$1" pin="1"/>
-<pinref part="GND31" gate="1" pin="GND"/>
-</segment>
-<segment>
 <pinref part="SW2" gate="G$1" pin="2"/>
 <pinref part="GND13" gate="1" pin="GND"/>
@@
 <pinref part="C15" gate="G$1" pin="1"/>
 <pinref part="GND29" gate="1" pin="GND"/>
+</segment>
+<segment>
+<pinref part="C16" gate="G$1" pin="1"/>
+<pinref part="GND31" gate="1" pin="GND"/>
 </segment>
 </net>
@@
 </segment>
 </net>
-<net name="N$21" class="0">
-<segment>
-<pinref part="C16" gate="G$1" pin="2"/>
-<pinref part="C17" gate="G$1" pin="1"/>
-</segment>
-</net>
 <net name="N$15" class="0">
 <segment>
@@
 <junction x="91.44" y="2.54"/>
 <wire x1="185.42" y1="-10.16" x2="185.42" y2="27.94" width="0.1524" layer="91"/>
-<pinref part="C17" gate="G$1" pin="2"/>
 <wire x1="165.1" y1="27.94" x2="170.18" y2="27.94" width="0.1524" layer="91"/>
 <pinref part="C13" gate="G$1" pin="2"/>
 <junction x="165.1" y="27.94"/>
 <wire x1="170.18" y1="27.94" x2="175.26" y2="27.94" width="0.1524" layer="91"/>
-<wire x1="175.26" y1="27.94" x2="180.34" y2="27.94" width="0.1524" layer="91"/>
 <wire x1="160.02" y1="27.94" x2="165.1" y2="27.94" width="0.1524" layer="91"/>
 <pinref part="C12" gate="G$1" pin="2"/>
@@
 <junction x="175.26" y="27.94"/>
 <wire x1="185.42" y1="27.94" x2="180.34" y2="27.94" width="0.1524" layer="91"/>
+<pinref part="C16" gate="G$1" pin="2"/>
+<wire x1="180.34" y1="27.94" x2="175.26" y2="27.94" width="0.1524" layer="91"/>
 <junction x="180.34" y="27.94"/>
 </segment>

Commit message: add
Parts:
- removed C21: (no value), myparts:CAPACITOR-0603
- added C17: (no value), myparts:CAPACITOR-0603
Connections:
- net GND: now also C17.1; no longer C21.1
- net N$14: now also C20.2; no longer C21.2
- net N$2: now also C17.2; no longer C18.2
- net N$20: now also C18.2; no longer C19.2
- net N$25: now also C19.2; no longer C20.2
Other:
- moved on the sheet: C18, C19, C20
Changed lines of the file:
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@@
 <setting verticaltext="up"/>
 </settings>
-<grid distance="0.1" unitdist="inch" unit="inch" style="lines" multiple="1" display="no" altdistance="0.01" altunitdist="inch" altunit="inch"/>
+<grid distance="0.02" unitdist="inch" unit="inch" style="lines" multiple="1" display="no" altdistance="0.01" altunitdist="inch" altunit="inch"/>
 <layers>
 <layer number="1" name="Top" color="4" fill="1" visible="no" active="no"/>
@@
 <part name="R10" library="myparts" deviceset="RESISTOR-0603" device=""/>
 <part name="GND7" library="myparts" deviceset="GND" device=""/>
-<part name="C18" library="myparts" deviceset="CAPACITOR-0603" device=""/>
+<part name="C17" library="myparts" deviceset="CAPACITOR-0603" device=""/>
 <part name="CON3" library="myparts" deviceset="SMA-RF" device=""/>
 <part name="GND8" library="myparts" deviceset="GND" device=""/>
@@
 <part name="R16" library="myparts" deviceset="RESISTOR-0603" device=""/>
 <part name="GND53" library="myparts" deviceset="GND" device=""/>
-<part name="C19" library="myparts" deviceset="CAPACITOR-0603" device=""/>
+<part name="C18" library="myparts" deviceset="CAPACITOR-0603" device=""/>
 <part name="GND54" library="myparts" deviceset="GND" device=""/>
 <part name="Q1" library="myparts" deviceset="P-MOSFET" device=""/>
@@
 <part name="R13" library="myparts" deviceset="RESISTOR-0603" device=""/>
 <part name="R14" library="myparts" deviceset="RESISTOR-0603" device=""/>
+<part name="C19" library="myparts" deviceset="CAPACITOR-0603" device=""/>
 <part name="C20" library="myparts" deviceset="CAPACITOR-0603" device=""/>
-<part name="C21" library="myparts" deviceset="CAPACITOR-0603" device=""/>
 <part name="GND26" library="myparts" deviceset="GND" device=""/>
 <part name="GND27" library="myparts" deviceset="GND" device=""/>
@@
 <attribute name="VALUE" x="152.4" y="-8.128" size="1.778" layer="96"/>
 </instance>
-<instance part="C18" gate="G$1" x="154.94" y="-2.54" smashed="yes" rot="R90">
+<instance part="C17" gate="G$1" x="154.94" y="-2.54" smashed="yes" rot="R90">
 <attribute name="NAME" x="157.988" y="1.778" size="1.778" layer="95" rot="R90" align="center-left"/>
 <attribute name="VALUE" x="150.114" y="1.27" size="1.778" layer="96" rot="R90" align="center-left"/>
@@
 <attribute name="VALUE" x="-58.42" y="9.652" size="1.778" layer="96"/>
 </instance>
-<instance part="C19" gate="G$1" x="-50.8" y="15.24" smashed="yes" rot="R90">
-<attribute name="NAME" x="-53.848" y="19.05" size="1.778" layer="95" rot="R90" align="center-left"/>
+<instance part="C18" gate="G$1" x="-50.8" y="15.24" smashed="yes" rot="R90">
+<attribute name="NAME" x="-47.752" y="19.05" size="1.778" layer="95" rot="R90" align="center-left"/>
 <attribute name="VALUE" x="-55.626" y="19.05" size="1.778" layer="96" rot="R90" align="center-left"/>
 </instance>
@@
 <attribute name="VALUE" x="-82.55" y="-18.288" size="1.778" layer="96" rot="R270" align="center-left"/>
 </instance>
-<instance part="C20" gate="G$1" x="-81.28" y="-15.24" smashed="yes" rot="R270">
+<instance part="C19" gate="G$1" x="-81.28" y="-15.24" smashed="yes" rot="R270">
 <attribute name="NAME" x="-80.264" y="-23.114" size="1.778" layer="95" rot="R270" align="center-left"/>
 <attribute name="VALUE" x="-76.454" y="-19.05" size="1.778" layer="96" rot="R270" align="center-left"/>
 </instance>
-<instance part="C21" gate="G$1" x="-76.2" y="-15.24" smashed="yes" rot="R270">
+<instance part="C20" gate="G$1" x="-76.2" y="-15.24" smashed="yes" rot="R270">
 <attribute name="NAME" x="-75.184" y="-23.114" size="1.778" layer="95" rot="R270" align="center-left"/>
 <attribute name="VALUE" x="-71.374" y="-19.05" size="1.778" layer="96" rot="R270" align="center-left"/>
@@
 </instance>
 <instance part="C16" gate="G$1" x="180.34" y="15.24" smashed="yes" rot="R90">
-<attribute name="NAME" x="177.292" y="19.05" size="1.778" layer="95" rot="R90" align="center-left"/>
+<attribute name="NAME" x="179.324" y="15.494" size="1.778" layer="95" rot="R90" align="center-left"/>
 <attribute name="VALUE" x="175.514" y="19.05" size="1.778" layer="96" rot="R90" align="center-left"/>
 </instance>
@@
 <net name="GND" class="0">
 <segment>
-<pinref part="C18" gate="G$1" pin="1"/>
+<pinref part="C17" gate="G$1" pin="1"/>
 <pinref part="GND7" gate="1" pin="GND"/>
 </segment>
@@
 </segment>
 <segment>
-<pinref part="C19" gate="G$1" pin="1"/>
+<pinref part="C18" gate="G$1" pin="1"/>
 <pinref part="GND54" gate="1" pin="GND"/>
 </segment>
@@
 </segment>
 <segment>
+<pinref part="C19" gate="G$1" pin="1"/>
+<pinref part="GND27" gate="1" pin="GND"/>
+</segment>
+<segment>
 <pinref part="C20" gate="G$1" pin="1"/>
-<pinref part="GND27" gate="1" pin="GND"/>
-</segment>
-<segment>
-<pinref part="C21" gate="G$1" pin="1"/>
 <pinref part="GND28" gate="1" pin="GND"/>
 </segment>
@@
 <segment>
 <pinref part="R10" gate="G$1" pin="1"/>
-<pinref part="C18" gate="G$1" pin="2"/>
+<pinref part="C17" gate="G$1" pin="2"/>
 <junction x="154.94" y="10.16"/>
 <pinref part="R9" gate="G$1" pin="1"/>
@@
 <wire x1="-55.88" y1="27.94" x2="-55.88" y2="33.02" width="0.1524" layer="91"/>
 <pinref part="R15" gate="G$1" pin="2"/>
-<pinref part="C19" gate="G$1" pin="2"/>
+<pinref part="C18" gate="G$1" pin="2"/>
 <pinref part="IC1" gate="G$1" pin="ADC6/PF6"/>
 <wire x1="-55.88" y1="33.02" x2="-55.88" y2="35.56" width="0.1524" layer="91"/>
@@
 <wire x1="-71.12" y1="-40.64" x2="-88.9" y2="-40.64" width="0.1524" layer="91"/>
 <junction x="-88.9" y="-40.64"/>
-<pinref part="C21" gate="G$1" pin="2"/>
+<pinref part="C20" gate="G$1" pin="2"/>
 <wire x1="-76.2" y1="-27.94" x2="-76.2" y2="-33.02" width="0.1524" layer="91"/>
 <wire x1="-76.2" y1="-33.02" x2="-88.9" y2="-33.02" width="0.1524" layer="91"/>
@@
 <wire x1="-73.66" y1="-43.18" x2="-86.36" y2="-43.18" width="0.1524" layer="91"/>
 <junction x="-86.36" y="-43.18"/>
-<pinref part="C20" gate="G$1" pin="2"/>
+<pinref part="C19" gate="G$1" pin="2"/>
 <wire x1="-81.28" y1="-27.94" x2="-81.28" y2="-30.48" width="0.1524" layer="91"/>
 <wire x1="-81.28" y1="-30.48" x2="-86.36" y2="-30.48" width="0.1524" layer="91"/>

Commit message: init
Parts:
- added D2: (no value), myparts:ZENER-SOD123
- added Q2: (no value), myparts:P-MOSFET
- added R17, R18, R19: (no value), myparts:RESISTOR-0603
Connections:
- new net N$21: D2.K, Q2.G, R17.2, R18.2
- new net N$26: Q1.S, Q2.S, R19.2
- net GND: now also D2.A, R18.1
- net UVCC: now also R17.1
- net VCC: now also Q2.D, R19.1; no longer Q1.S
Other:
- moved on the sheet: BAT1, J1, Q1
Changed lines of the file:
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@@
 <part name="GND5" library="myparts" deviceset="GND" device=""/>
 <part name="GND6" library="myparts" deviceset="GND" device=""/>
-<part name="SUP2" library="myparts" deviceset="VCC" device=""/>
 <part name="R15" library="myparts" deviceset="RESISTOR-0603" device=""/>
 <part name="IC2" library="myparts" deviceset="VREG-SOT23-3" device=""/>
@@
 <part name="GND29" library="myparts" deviceset="GND" device=""/>
 <part name="C16" library="myparts" deviceset="CAPACITOR-10-5" device=""/>
+<part name="R17" library="myparts" deviceset="RESISTOR-0603" device=""/>
+<part name="R18" library="myparts" deviceset="RESISTOR-0603" device=""/>
+<part name="Q2" library="myparts" deviceset="P-MOSFET" device=""/>
+<part name="D2" library="myparts" deviceset="ZENER-SOD123" device=""/>
+<part name="U$4" library="myparts" deviceset="UVCC" device=""/>
+<part name="GND30" library="myparts" deviceset="GND" device=""/>
+<part name="GND32" library="myparts" deviceset="GND" device=""/>
+<part name="SUP2" library="myparts" deviceset="VCC" device=""/>
+<part name="R19" library="myparts" deviceset="RESISTOR-0603" device=""/>
+<part name="SUP10" library="myparts" deviceset="VCC" device=""/>
 </parts>
 <sheets>
@@
 <attribute name="VALUE" x="-53.34" y="9.652" size="1.778" layer="96"/>
 </instance>
-<instance part="Q1" gate="G$1" x="-127" y="7.62" smashed="yes" rot="MR90">
-<attribute name="NAME" x="-122.936" y="14.224" size="1.778" layer="95" rot="MR0" align="center-left"/>
-<attribute name="VALUE" x="-125.222" y="13.208" size="1.778" layer="96" rot="MR90" align="center-left"/>
-</instance>
-<instance part="GND52" gate="1" x="-121.92" y="5.08" smashed="yes">
-<attribute name="VALUE" x="-124.46" y="2.032" size="1.778" layer="96"/>
+<instance part="Q1" gate="G$1" x="-142.24" y="-17.78" smashed="yes" rot="MR90">
+<attribute name="NAME" x="-138.176" y="-11.176" size="1.778" layer="95" rot="MR0" align="center-left"/>
+<attribute name="VALUE" x="-140.462" y="-12.192" size="1.778" layer="96" rot="MR90" align="center-left"/>
+</instance>
+<instance part="GND52" gate="1" x="-137.16" y="-35.56" smashed="yes">
+<attribute name="VALUE" x="-139.7" y="-38.608" size="1.778" layer="96"/>
 </instance>
 <instance part="R5" gate="G$1" x="86.36" y="10.16" smashed="yes" rot="R90">
@@
 <attribute name="VALUE" x="-40.386" y="-48.006" size="1.778" layer="96" align="center-left"/>
 </instance>
-<instance part="BAT1" gate="G$1" x="-142.24" y="12.7" smashed="yes" rot="R270">
-<attribute name="NAME" x="-145.288" y="9.144" size="1.778" layer="95" rot="R270" align="center-left"/>
-<attribute name="VALUE" x="-137.414" y="8.89" size="1.778" layer="96" rot="R270" align="center-left"/>
-</instance>
-<instance part="GND67" gate="1" x="-142.24" y="-2.54" smashed="yes">
-<attribute name="VALUE" x="-144.78" y="-5.588" size="1.778" layer="96"/>
+<instance part="BAT1" gate="G$1" x="-157.48" y="-12.7" smashed="yes" rot="R270">
+<attribute name="NAME" x="-160.528" y="-16.256" size="1.778" layer="95" rot="R270" align="center-left"/>
+<attribute name="VALUE" x="-152.654" y="-16.51" size="1.778" layer="96" rot="R270" align="center-left"/>
+</instance>
+<instance part="GND67" gate="1" x="-157.48" y="-35.56" smashed="yes">
+<attribute name="VALUE" x="-160.02" y="-38.608" size="1.778" layer="96"/>
 </instance>
 <instance part="F1" gate="G$1" x="-132.08" y="33.02" smashed="yes">
@@
 <attribute name="VALUE" x="-33.02" y="-66.548" size="1.778" layer="96"/>
 </instance>
-<instance part="J1" gate="G$1" x="-129.54" y="12.7" smashed="yes" rot="R180">
-<attribute name="NAME" x="-134.62" y="10.668" size="1.778" layer="95" rot="R180" align="center-left"/>
-<attribute name="VALUE" x="-132.588" y="8.89" size="1.778" layer="96" rot="R180" align="center-left"/>
+<instance part="J1" gate="G$1" x="-144.78" y="-12.7" smashed="yes" rot="R180">
+<attribute name="NAME" x="-149.86" y="-14.732" size="1.778" layer="95" rot="R180" align="center-left"/>
+<attribute name="VALUE" x="-147.828" y="-16.51" size="1.778" layer="96" rot="R180" align="center-left"/>
 </instance>
 <instance part="SW2" gate="G$1" x="-48.26" y="-48.26" smashed="yes" rot="R270">
@@
 <attribute name="VALUE" x="147.828" y="22.86" size="1.778" layer="96" rot="R90"/>
 </instance>
-<instance part="SUP2" gate="G$1" x="-119.38" y="15.24" smashed="yes">
-<attribute name="VALUE" x="-121.285" y="17.145" size="1.778" layer="96"/>
-</instance>
 <instance part="R15" gate="G$1" x="-55.88" y="48.26" smashed="yes" rot="R270">
 <attribute name="NAME" x="-57.912" y="44.196" size="1.778" layer="95" rot="R270" align="center-left"/>
@@
 <attribute name="NAME" x="179.324" y="15.494" size="1.778" layer="95" rot="R90" align="center-left"/>
 <attribute name="VALUE" x="175.514" y="19.05" size="1.778" layer="96" rot="R90" align="center-left"/>
+</instance>
+<instance part="R17" gate="G$1" x="-127" y="-33.02" smashed="yes" rot="R90">
+<attribute name="NAME" x="-128.524" y="-35.052" size="1.778" layer="95" rot="R90" align="center-left"/>
+<attribute name="VALUE" x="-130.81" y="-29.972" size="1.778" layer="96" rot="R90" align="center-left"/>
+</instance>
+<instance part="R18" gate="G$1" x="-124.46" y="-33.02" smashed="yes" rot="R90">
+<attribute name="NAME" x="-125.476" y="-35.052" size="1.778" layer="95" rot="R90" align="center-left"/>
+<attribute name="VALUE" x="-128.27" y="-29.972" size="1.778" layer="96" rot="R90" align="center-left"/>
+</instance>
+<instance part="Q2" gate="G$1" x="-116.84" y="-17.78" smashed="yes" rot="R90">
+<attribute name="NAME" x="-118.364" y="-11.176" size="1.778" layer="95" rot="R180" align="center-left"/>
+<attribute name="VALUE" x="-118.618" y="-12.192" size="1.778" layer="96" rot="R90" align="center-left"/>
+</instance>
+<instance part="D2" gate="G$1" x="-121.92" y="-20.32" smashed="yes" rot="R270">
+<attribute name="NAME" x="-122.936" y="-30.48" size="1.778" layer="95" rot="R270" align="center-left"/>
+<attribute name="VALUE" x="-118.11" y="-21.844" size="1.778" layer="96" rot="R270" align="center-left"/>
+</instance>
+<instance part="U$4" gate="G$1" x="-127" y="-35.56" smashed="yes" rot="R180">
+<attribute name="VALUE" x="-125.095" y="-37.465" size="1.778" layer="96" rot="R180"/>
+</instance>
+<instance part="GND30" gate="1" x="-124.46" y="-35.56" smashed="yes">
+<attribute name="VALUE" x="-127" y="-38.608" size="1.778" layer="96"/>
+</instance>
+<instance part="GND32" gate="1" x="-121.92" y="-35.56" smashed="yes">
+<attribute name="VALUE" x="-124.46" y="-38.608" size="1.778" layer="96"/>
+</instance>
+<instance part="SUP2" gate="G$1" x="-111.76" y="-10.16" smashed="yes">
+<attribute name="VALUE" x="-113.665" y="-8.255" size="1.778" layer="96"/>
+</instance>
+<instance part="R19" gate="G$1" x="-132.08" y="-33.02" smashed="yes" rot="R90">
+<attribute name="NAME" x="-133.604" y="-35.052" size="1.778" layer="95" rot="R90" align="center-left"/>
+<attribute name="VALUE" x="-135.89" y="-29.972" size="1.778" layer="96" rot="R90" align="center-left"/>
+</instance>
+<instance part="SUP10" gate="G$1" x="-132.08" y="-35.56" smashed="yes" rot="R180">
+<attribute name="VALUE" x="-130.175" y="-37.465" size="1.778" layer="96" rot="R180"/>
 </instance>
 </instances>
@@
 <pinref part="Q1" gate="G$1" pin="G"/>
 <pinref part="GND52" gate="1" pin="GND"/>
+<wire x1="-137.16" y1="-33.02" x2="-137.16" y2="-17.78" width="0.1524" layer="91"/>
 </segment>
 <segment>
 <pinref part="BAT1" gate="G$1" pin="-"/>
 <pinref part="GND67" gate="1" pin="GND"/>
+<wire x1="-157.48" y1="-33.02" x2="-157.48" y2="-25.4" width="0.1524" layer="91"/>
 </segment>
 <segment>
@@
 <pinref part="C16" gate="G$1" pin="1"/>
 <pinref part="GND31" gate="1" pin="GND"/>
+</segment>
+<segment>
+<pinref part="R18" gate="G$1" pin="1"/>
+<pinref part="GND30" gate="1" pin="GND"/>
+</segment>
+<segment>
+<pinref part="D2" gate="G$1" pin="A"/>
+<pinref part="GND32" gate="1" pin="GND"/>
 </segment>
 </net>
@@
 </segment>
 <segment>
-<pinref part="Q1" gate="G$1" pin="S"/>
+<pinref part="Q2" gate="G$1" pin="D"/>
 <pinref part="SUP2" gate="G$1" pin="VCC"/>
+<wire x1="-114.3" y1="-12.7" x2="-111.76" y2="-12.7" width="0.1524" layer="91"/>
+</segment>
+<segment>
+<pinref part="R19" gate="G$1" pin="1"/>
+<pinref part="SUP10" gate="G$1" pin="VCC"/>
 </segment>
 </net>
@@
 <junction x="-119.38" y="33.02"/>
 <junction x="-109.22" y="33.02"/>
+</segment>
+<segment>
+<pinref part="R17" gate="G$1" pin="1"/>
+<pinref part="U$4" gate="G$1" pin="UVCC"/>
 </segment>
 </net>
@@
 </segment>
 </net>
+<net name="N$21" class="0">
+<segment>
+<pinref part="R17" gate="G$1" pin="2"/>
+<pinref part="R18" gate="G$1" pin="2"/>
+<wire x1="-127" y1="-20.32" x2="-124.46" y2="-20.32" width="0.1524" layer="91"/>
+<pinref part="D2" gate="G$1" pin="K"/>
+<wire x1="-124.46" y1="-20.32" x2="-121.92" y2="-20.32" width="0.1524" layer="91"/>
+<junction x="-124.46" y="-20.32"/>
+<pinref part="Q2" gate="G$1" pin="G"/>
+<wire x1="-121.92" y1="-17.78" x2="-121.92" y2="-20.32" width="0.1524" layer="91"/>
+<junction x="-121.92" y="-20.32"/>
+</segment>
+</net>
+<net name="N$26" class="0">
+<segment>
+<pinref part="Q1" gate="G$1" pin="S"/>
+<pinref part="Q2" gate="G$1" pin="S"/>
+<wire x1="-134.62" y1="-12.7" x2="-132.08" y2="-12.7" width="0.1524" layer="91"/>
+<pinref part="R19" gate="G$1" pin="2"/>
+<wire x1="-132.08" y1="-12.7" x2="-124.46" y2="-12.7" width="0.1524" layer="91"/>
+<wire x1="-132.08" y1="-20.32" x2="-132.08" y2="-12.7" width="0.1524" layer="91"/>
+<junction x="-132.08" y="-12.7"/>
+</segment>
+</net>
